File: esp-car-3.0/esp-car.kicad_pcb (KiCad board)
At the start: 2 copper layers, 113 x 120.5 mm, 36 parts, among them J1 Conn_01x07_Socket, J2 Conn_01x07_Socket, U1 ESP32-DEVKIT-V1, U3 L293D

Commit message: finalizado, tem que revisar, esp_car_3.3
revisa os pinos e muda, trabalhe com o stevan vitor
Parts:
- ALI1, MotorD1, MotorE1: footprint IFSUL Camaquã:TerminalBlock_Phoenix_MKDS-1,5-2-5.08_1x02_P5.08mm_Horizontal -> Connector_PinSocket_2.54mm:PinSocket_1x02_P2.54mm_Vertical
- moved C1 14.8 mm to (128.5, 119.9)
- moved TelaOLED1 1.56 mm to (173.1, 126.6)
- moved giroscopio1 1.56 mm to (177.6, 131.7)
- moved MotorE1 1.33 mm to (155.2, 132.6), turned to 90 degrees
- moved R8 0.96 mm to (163.0, 42.5)
- moved ALI1 0.29 mm to (173.2, 138.8), turned to 90 degrees
- turned MotorD1 to -90 degrees
Connections:
- U1 pad 21: unconnected-(U1-D32-Pad21) -> INF_TD
- U1 pad 24: IN3 -> unconnected-(U1-D26-Pad24)
- U1 pad 8: unconnected-(U1-D5-Pad8) -> IN3
Routing:
- net SDA: track 4.50 -> 199.0 mm, vias 0 -> 3
- net 3v3: track 0.00 -> 161.8 mm, vias 0 -> 11
- net GND: track 0.00 -> 155.5 mm, vias 0 -> 8
- net SCL: track 4.50 -> 137.6 mm, vias 0 -> 5
- net INF_FE: track 0.00 -> 85.9 mm
- net LD: track 0.00 -> 69.6 mm
- net INF_FD: track 0.00 -> 57.8 mm
- net IN2: track 0.00 -> 55.0 mm, vias 0 -> 2
- net LE: track 0.00 -> 48.2 mm
- net IN3: track 0.00 -> 47.6 mm
- net INF_TD: track 0.00 -> 43.7 mm, vias 0 -> 2
- net INF_C: track 0.00 -> 39.9 mm, vias 0 -> 2
- net CD: track 0.00 -> 39.3 mm
- net CE: track 0.00 -> 37.3 mm
- net OUTE: track 0.00 -> 34.8 mm
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
Commit message: finalizada agora
Connections:
- U1 pad 17: LE -> unconnected-(U1-VP-Pad17)
- U1 pad 18: CE -> unconnected-(U1-VN-Pad18)
- U1 pad 20: unconnected-(U1-D35-Pad20) -> LE
- U1 pad 23: unconnected-(U1-D25-Pad23) -> CE
Routing:
- net LE: track 48.2 -> 66.6 mm
- net CE: track 37.3 -> 53.3 mm
- net INF_C: track 39.9 -> 46.9 mm
- net OUTD: track 26.4 -> 28.2 mm
- net LD: track 69.6 -> 71.2 mm
- net SDA: track 199.0 -> 198.2 mm
- net INF_FD: track 57.8 -> 57.2 mm

Commit message: versão finalizada e polida
muitas alterações
Parts:
- added C2: C, Capacitor_THT:CP_Radial_D10.0mm_P3.50mm, F.Cu at (167.4, 133.4)
- added extra2: Conn_01x01_Socket, Connector_PinSocket_2.54mm:PinSocket_1x01_P2.54mm_Vertical, F.Cu at (183.8, 110.0)
- moved R4 4.48 mm to (199.5, 29.8)
- moved R8 4.25 mm to (159.5, 45.0), turned to 90 degrees
- moved R6 3.70 mm to (142.2, 39.8), turned to 90 degrees
- moved ALI1 3.23 mm to (170.5, 140.5), turned to -90 degrees
- moved BotaoRotatorio1 3.18 mm to (179.9, 109.7)
- moved EN1 2.26 mm to (118.7, 59.0)
- moved LED1 1.72 mm to (131.2, 108.7)
- moved R220 1.72 mm to (127.0, 111.2)
- moved C1 1.55 mm to (127.0, 119.5)
- moved BZ1 0.79 mm to (138.5, 128.0)
Connections:
- J1 pad 5: 3v3 -> C1
- J2 pad 5: 3v3 -> C2
- U1 pad 18: unconnected-(U1-VN-Pad18) -> LE
- U1 pad 20: LE -> C1
- U1 pad 24: unconnected-(U1-D26-Pad24) -> C2
- U1 pad 4: unconnected-(U1-D2-Pad4) -> 2
Routing:
- net SCL: track 137.6 -> 278.4 mm
- net SDA: track 198.2 -> 334.7 mm, vias 3 -> 4
- net C2: track 0.00 -> 112.2 mm, vias 0 -> 1
- net C1: track 0.00 -> 60.8 mm, vias 0 -> 1
- net 3v3: track 161.8 -> 216.9 mm, vias 11 -> 10
- net 2: track 0.00 -> 43.3 mm, vias 0 -> 2
- net GND: track 155.5 -> 178.2 mm, vias 8 -> 7
- net LED: track 29.6 -> 45.2 mm
- net CE: track 53.3 -> 62.7 mm
- net LE: track 66.6 -> 60.4 mm
- net INF_TD: track 44.1 -> 50.2 mm
- net Net-(LINHA_DIR1-PadA): track 3.39 -> 8.02 mm
- net OUTE: track 34.8 -> 38.4 mm
- net S2: track 30.0 -> 27.5 mm
- net S1: track 23.9 -> 21.3 mm
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